File: kikad/TZXDuino.kicad_pcb (KiCad board)
At the start: 2 copper layers, 97.8 x 82.5 mm, 19 parts, among them J1 SPECCY, J2 SPEAKER, J3 POWER IN, SW1 CHERRY MX, SW2 CHERRY MX, SW3 CHERRY MX, SW4 CHERRY MX, U1 ARDUINO NANO, U2 LCD 1602, U3 Catalex_Micro_SD

Commit message: Fixing
Parts:
- removed H1, H2, H3, H4: MountingHole, MountingHole:MountingHole_3mm_Pad
- removed MISO, MOSI, SCK: SolderJumper-2_P1.3mm_Open_RoundedPad1.0x1.5mm, Jumper:SolderJumper-2_P1.3mm_Open_RoundedPad1.0x1.5mm
- removed U3: Catalex_Micro_SD, TZXDuino:Catalex_Micro_SD
- added J4: SD_Card, TZXduino_beta:SDCARD_4UCONN, F.Cu at (129.9, 103.9)
- added R2: 2.2K, Resistor_THT:R_Axial_DIN0207_L6.3mm_D2.5mm_P10.16mm_Horizontal, F.Cu at (112.4, 93.0)
- added R3: 2.2K, Resistor_THT:R_Axial_DIN0207_L6.3mm_D2.5mm_P10.16mm_Horizontal, F.Cu at (112.5, 110.5)
- added R4: 2.2K, Resistor_THT:R_Axial_DIN0207_L6.3mm_D2.5mm_P10.16mm_Horizontal, F.Cu at (98.1, 106.8)
- added R5: 3.3K, Resistor_THT:R_Axial_DIN0207_L6.3mm_D2.5mm_P10.16mm_Horizontal, F.Cu at (122.3, 96.6)
- added R6: 3.3K, Resistor_THT:R_Axial_DIN0207_L6.3mm_D2.5mm_P10.16mm_Horizontal, F.Cu at (117.6, 106.8)
- added R7: 3.3K, Resistor_THT:R_Axial_DIN0207_L6.3mm_D2.5mm_P10.16mm_Horizontal, F.Cu at (112.9, 106.9)
- added R8: 10K, Resistor_THT:R_Axial_DIN0207_L6.3mm_D2.5mm_P10.16mm_Horizontal, F.Cu at (104.5, 102.0)
- moved SW1 19.8 mm to (60.1, 126.7)
- moved SW2 19.8 mm to (80.4, 126.7)
- moved SW3 19.8 mm to (100.7, 126.7)
- moved SW4 19.8 mm to (121.1, 126.7)
Connections:
- J1 pad TN: Net-(J1-PadTN) -> unconnected-(J1-PadTN)
- U1 pad 1: Net-(U1-Pad1) -> unconnected-(U1-D1/TX-Pad1)
- U1 pad 17: Net-(U1-Pad17) -> +3.3V
- U1 pad 18: Net-(U1-Pad18) -> unconnected-(U1-AREF-Pad18)
- U1 pad 2: Net-(U1-Pad2) -> unconnected-(U1-D0/RX-Pad2)
- U1 pad 23: Net-(U1-Pad23) -> unconnected-(U1-A4-Pad23)
- U1 pad 24: Net-(U1-Pad24) -> unconnected-(U1-A5-Pad24)
- U1 pad 25: Net-(U1-Pad25) -> unconnected-(U1-A6-Pad25)
- U1 pad 26: Net-(U1-Pad26) -> unconnected-(U1-A7-Pad26)
- U1 pad 28: Net-(U1-Pad28) -> unconnected-(U1-~{RESET}-Pad28)
- U1 pad 3: Net-(U1-Pad3) -> unconnected-(U1-~{RESET}-Pad3)
- U2 pad 10: Net-(U2-Pad10) -> unconnected-(U2-D3-Pad10)
- U2 pad 7: Net-(U2-Pad7) -> unconnected-(U2-D0-Pad7)
- U2 pad 8: Net-(U2-Pad8) -> unconnected-(U2-D1-Pad8)
- U2 pad 9: Net-(U2-Pad9) -> unconnected-(U2-D2-Pad9)
Routing:
- net +5V: track 112.8 -> 0.00 mm
- net CS: track 77.8 -> 0.00 mm
- net MOSI: track 74.7 -> 0.00 mm
- net A3: track 73.4 -> 0.00 mm
- net MISO: track 59.0 -> 0.00 mm
- net SCK: track 56.9 -> 0.00 mm
- net A2: track 55.6 -> 0.00 mm
- net D5: track 49.7 -> 0.00 mm
- net D4: track 49.7 -> 0.00 mm
- net D3: track 49.7 -> 0.00 mm
- net D2: track 49.7 -> 0.00 mm
- net D6: track 45.5 -> 0.00 mm
- net D7: track 44.5 -> 0.00 mm
- net A1: track 37.8 -> 0.00 mm
- net Net-(J3-Pin_2): track 36.3 -> 0.00 mm
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- removed copper zone on B.Cu, net GND
Other:
- board outline removed
- board text removed: "MICRO SD"

Commit message: Update
Parts:
- removed BOARD: PROTOBOARD, TZXDuino:ProtoBoard
- moved J2 8.57 mm to (54.1, 69.7)
Changed lines of the file:
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@@
     (fp_arc (start 63.7 8) (mid 64.053553 8.146447) (end 64.2 8.5)
       (stroke (width 0.12) (type solid)) (layer "F.SilkS"))
-    (fp_arc (start 64.20104 22.49932) (mid 64.054473 22.853115) (end 63.70066 22.9997)
+    (fp_arc (start 64.20104 22.49932) (mid 64.054479 22.85315) (end 63.70066 22.9997)
       (stroke (width 0.12) (type solid)) (layer "F.SilkS"))
     (fp_line (start -8.25 -2.75) (end -8.25 33.75)
@@
     )
   )
-  (footprint "TZXDuino:ProtoBoard" (layer "F.Cu")
-    (at 54.61 59.69)
-    (descr "Through hole straight pin header, 1x06, 2.54mm pitch, single row")
-    (tags "Through hole pin header THT 1x06 2.54mm single row")
-    (attr through_hole)
-    (fp_text reference "BOARD" (at 8.636 -2.032) (layer "F.SilkS")
-        (effects (font (size 1 1) (thickness 0.15)))
-    )
-    (fp_text value "PROTOBOARD" (at 6.35 -0.254 180) (layer "F.Fab")
-        (effects (font (size 1 1) (thickness 0.15)))
-    )
-    (fp_line (start -1.33 -1.27) (end -1.33 11.49)
-      (stroke (width 0.12) (type solid)) (layer "F.SilkS"))
-    (fp_line (start -1.33 -1.27) (end 11.43 -1.27)
-      (stroke (width 0.12) (type solid)) (layer "F.SilkS"))
-    (fp_line (start -1.33 11.49) (end 11.43 11.49)
-      (stroke (width 0.12) (type solid)) (layer "F.SilkS"))
-    (fp_line (start 11.43 -1.27) (end 11.43 11.49)
-      (stroke (width 0.12) (type solid)) (layer "F.SilkS"))
-    (pad "" thru_hole circle (at 0 0) (size 1.7 1.7) (drill 1) (layers "*.Cu" "*.Mask"))
-    (pad "" thru_hole oval (at 0 2.54) (size 1.7 1.7) (drill 1) (layers "*.Cu" "*.Mask"))
-    (pad "" thru_hole oval (at 0 5.08) (size 1.7 1.7) (drill 1) (layers "*.Cu" "*.Mask"))
-    (pad "" thru_hole oval (at 0 7.62) (size 1.7 1.7) (drill 1) (layers "*.Cu" "*.Mask"))
-    (pad "" thru_hole oval (at 0 10.16) (size 1.7 1.7) (drill 1) (layers "*.Cu" "*.Mask"))
-    (pad "" thru_hole circle (at 2.54 0) (size 1.7 1.7) (drill 1) (layers "*.Cu" "*.Mask"))
-    (pad "" thru_hole oval (at 2.54 2.54) (size 1.7 1.7) (drill 1) (layers "*.Cu" "*.Mask"))
-    (pad "" thru_hole oval (at 2.54 5.08) (size 1.7 1.7) (drill 1) (layers "*.Cu" "*.Mask"))
-    (pad "" thru_hole oval (at 2.54 7.62) (size 1.7 1.7) (drill 1) (layers "*.Cu" "*.Mask"))
-    (pad "" thru_hole oval (at 2.54 10.16) (size 1.7 1.7) (drill 1) (layers "*.Cu" "*.Mask"))
-    (pad "" thru_hole circle (at 5.08 0) (size 1.7 1.7) (drill 1) (layers "*.Cu" "*.Mask"))
-    (pad "" thru_hole oval (at 5.08 2.54) (size 1.7 1.7) (drill 1) (layers "*.Cu" "*.Mask"))
-    (pad "" thru_hole oval (at 5.08 5.08) (size 1.7 1.7) (drill 1) (layers "*.Cu" "*.Mask"))
-    (pad "" thru_hole oval (at 5.08 7.62) (size 1.7 1.7) (drill 1) (layers "*.Cu" "*.Mask"))
-    (pad "" thru_hole oval (at 5.08 10.16) (size 1.7 1.7) (drill 1) (layers "*.Cu" "*.Mask"))
-    (pad "" thru_hole circle (at 7.62 0) (size 1.7 1.7) (drill 1) (layers "*.Cu" "*.Mask"))
-    (pad "" thru_hole oval (at 7.62 2.54) (size 1.7 1.7) (drill 1) (layers "*.Cu" "*.Mask"))
-    (pad "" thru_hole oval (at 7.62 5.08) (size 1.7 1.7) (drill 1) (layers "*.Cu" "*.Mask"))
-    (pad "" thru_hole oval (at 7.62 7.62) (size 1.7 1.7) (drill 1) (layers "*.Cu" "*.Mask"))
-    (pad "" thru_hole oval (at 7.62 10.16) (size 1.7 1.7) (drill 1) (layers "*.Cu" "*.Mask"))
-    (pad "" thru_hole circle (at 10.16 0) (size 1.7 1.7) (drill 1) (layers "*.Cu" "*.Mask"))
-    (pad "" thru_hole oval (at 10.16 2.54) (size 1.7 1.7) (drill 1) (layers "*.Cu" "*.Mask"))
-    (pad "" thru_hole oval (at 10.16 5.08) (size 1.7 1.7) (drill 1) (layers "*.Cu" "*.Mask"))
-    (pad "" thru_hole oval (at 10.16 7.62) (size 1.7 1.7) (drill 1) (layers "*.Cu" "*.Mask"))
-    (pad "" thru_hole oval (at 10.16 10.16) (size 1.7 1.7) (drill 1) (layers "*.Cu" "*.Mask"))
-  )
   (footprint "Connector_PinHeader_2.54mm:PinHeader_1x02_P2.54mm_Vertical" (layer "F.Cu")
-    (at 62.23 72.39 90)
+    (at 54.097 69.6976 90)
     (descr "Through hole straight pin header, 1x02, 2.54mm pitch, single row")
     (tags "Through hole pin header THT 1x02 2.54mm single row")

Commit message: Update
Parts:
- removed J4: SD_Card, TZXduino_beta:SDCARD_4UCONN
- added J5: Jack_3.5mm_5pin, TZXduino_beta:audiojack_5_pin, B.Cu at (89.1, 102.9)
- J1: value SPECCY -> SD_Card; footprint TZXDuino:PJ-316 -> TZXduino_beta:SDCARD_4UCONN; moved to B.Cu
- J2: footprint Connector_PinHeader_2.54mm:PinHeader_1x02_P2.54mm_Vertical -> TZXduino_beta:Speaker; moved to B.Cu
- J3: value POWER IN -> Conn_01x04_Pin; footprint TZXDuino:PinHeader_1x02_P2.54mm_Horizontal -> TZXduino_beta:USB-C Power board; moved to B.Cu
- R1: footprint Resistor_THT:R_Axial_DIN0204_L3.6mm_D1.6mm_P7.62mm_Horizontal -> Resistor_THT:R_Axial_DIN0207_L6.3mm_D2.5mm_P10.16mm_Horizontal; moved to B.Cu
- R2, R3, R4, R5, R6, R7, R8, U1: moved to B.Cu
- moved J2 125.7 mm to (175.0, 104.2)
- moved J3 118.0 mm to (176.7, 118.0), turned to -90 degrees
- moved J1 93.1 mm to (146.7, 82.2), turned to 0 degrees
- moved R1 81.4 mm to (132.9, 101.0), turned to 0 degrees
- moved SW4 44.2 mm to (161.7, 109.3)
- moved SW2 44.0 mm to (120.8, 109.2)
- moved SW1 44.0 mm to (100.5, 109.2)
- moved SW3 44.0 mm to (141.1, 109.2)
- moved U1 43.2 mm to (133.6, 89.6), turned to 90 degrees
- moved R8 29.4 mm to (132.9, 94.4), turned to 0 degrees
- moved U2 25.7 mm to (96.5, 69.6)
- moved R3 16.1 mm to (102.7, 97.8)
- moved R4 13.3 mm to (102.7, 94.3)
- moved R7 13.0 mm to (116.6, 94.4), turned to 0 degrees
- moved R2 12.8 mm to (102.7, 101.2)
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Connections:
- J3 pad 1: GND -> Net-(J3-Pin_1)
- J3 pad 2: Net-(J3-Pin_2) -> unconnected-(J3-Pin_2-Pad2)
- R2 pad 2: Net-(J4-VSS-Pad3) -> Net-(J1-CLK)
- R3 pad 2: Net-(J4-VSS-Pad6) -> Net-(J1-CMD)
- R4 pad 2: Net-(J4-DAT0) -> Net-(J1-CD/DAT3)
- R5 pad 1: Net-(J4-VSS-Pad3) -> Net-(J1-CLK)
- R6 pad 1: Net-(J4-VSS-Pad6) -> Net-(J1-CMD)
- R7 pad 1: Net-(J4-DAT0) -> Net-(J1-CD/DAT3)
- U1 pad 30: Net-(J3-Pin_2) -> Net-(J3-Pin_1)
Routing:
- net GND: track 0.00 -> 255.6 mm
- net MISO: track 0.00 -> 85.3 mm
- net D5: track 0.00 -> 84.4 mm
- net D7: track 0.00 -> 75.1 mm
- net +3.3V: track 0.00 -> 73.3 mm
- net D8: track 0.00 -> 73.0 mm
- net Net-(U2-VO): track 0.00 -> 69.0 mm, vias 0 -> 1
- net Net-(J3-Pin_1): track 0.00 -> 68.2 mm, vias 0 -> 1
- net A1: track 0.00 -> 66.1 mm, vias 0 -> 1
- net A3: track 0.00 -> 62.9 mm, vias 0 -> 1
- net +5V: track 0.00 -> 57.0 mm, vias 0 -> 2
- net A2: track 0.00 -> 55.7 mm, vias 0 -> 1
- net D4: track 0.00 -> 54.3 mm, vias 0 -> 2
- net Net-(J1-CLK): track 0.00 -> 54.1 mm
- net Net-(J1-CD/DAT3): track 0.00 -> 47.2 mm
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Other:
- board outline added: 96.5 x 58.5 mm
- board text removed: "ARDUINO NANO"
- board text removed: "DESIGNED BY DENIS MALTSEV MADE IN USSR"
- board text removed: "GND"
- board text removed: "HTTPS://GITHUB.COM/MALTSEVDA/TZXDUINO_HF"
- board text removed: "LCD 1602"
- board text removed: "PIN CONFIG: BTN_PLAY - A2 BTN_STOP - A1 BTN_PREV - A0 BTN_NEXT - A3 LCD_RS - 7 LCD_EN - 6 LCD_D4 - 5 LCD_D5 - 4 LCD_D6 - 3 LCD_D7 - 2"
- board text removed: "POWER IN"
- board text removed: "SD_CHIPSELECT - 10 SND_SPEAKER - 8 SND_OUTPUT - 9"
- board text removed: "SPEAKER"
- board text removed: "SPECCY"

Commit message: Gerbers
Parts:
- added h1: MountingHole_2.5mm, MountingHole:MountingHole_2.5mm, F.Cu at (90.8, 69.3)
- added h2: MountingHole_2.5mm, MountingHole:MountingHole_2.5mm, F.Cu at (90.8, 100.8)
- added h3: MountingHole_2.5mm, MountingHole:MountingHole_2.5mm, F.Cu at (165.9, 100.6)
- moved J5 93.0 mm to (182.1, 99.5), turned to 180 degrees
- moved J2 24.1 mm to (150.9, 104.9), turned to 180 degrees
- moved SW4 3.56 mm to (158.1, 109.2)
- moved SW3 2.21 mm to (138.9, 109.2)
- moved SW2 1.10 mm to (119.7, 109.2)
- moved SW1 0.06 mm to (100.5, 109.2)
Routing:
- net D9: track 18.9 -> 73.0 mm
- net D7: track 75.1 -> 33.1 mm
- net A3: track 62.9 -> 98.0 mm
- net A2: track 55.7 -> 87.7 mm
- net D8: track 73.0 -> 48.9 mm
- net GND: track 255.6 -> 279.4 mm, vias 0 -> 1
- net D5: track 84.4 -> 64.2 mm, vias 0 -> 2
- net +3.3V: track 73.3 -> 60.7 mm, vias 0 -> 1
- net D2: track 46.3 -> 34.1 mm, vias 1 -> 0
- net A1: track 66.1 -> 55.9 mm, vias 1 -> 0
- net A0: track 40.3 -> 50.1 mm, vias 1 -> 0
- net Net-(J3-Pin_1): track 68.2 -> 76.8 mm
- net SCK: track 40.5 -> 32.4 mm
- net MISO: track 85.3 -> 90.5 mm
- net D4: track 54.3 -> 49.9 mm, vias 2 -> 1
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Other:
- board text added: "TZXDuino PCB by MadCat Ver.1.0 2024"
