File: kikad/TZXDuino.kicad_pcb (KiCad board)
At the start: 2 copper layers, 96.5 x 58.5 mm, 18 parts, among them J1 SD_Card, J2 SPEAKER, J3 Conn_01x04_Pin, J5 Jack_3.5mm_5pin, SW1 CHERRY MX, SW2 CHERRY MX, SW3 CHERRY MX, SW4 CHERRY MX, U1 ARDUINO NANO, U2 LCD 1602

Commit message: Update
Routing:
- net D5: track 84.4 -> 84.9 mm
Changed lines of the file:
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@@
   (segment (start 146.4248 94.1173) (end 134.0652 81.7577) (width 0.5) (layer "F.Cu") (net 21))
   (via (at 146.4248 94.1173) (size 1) (drill 0.5) (layers "F.Cu" "B.Cu") (net 21))
-  (segment (start 146.5429 94.1173) (end 161.6964 109.2708) (width 0.5) (layer "B.Cu") (net 21))
-  (segment (start 146.4248 94.1173) (end 146.5429 94.1173) (width 0.5) (layer "B.Cu") (net 21))
+  (segment (start 146.4248 94.1173) (end 147.0001 94.1173) (width 0.5) (layer "B.Cu") (net 21))
+  (segment (start 161.6964 108.8136) (end 161.6964 109.2708) (width 0.5) (layer "B.Cu") (net 21))
+  (segment (start 147.0001 94.1173) (end 161.6964 108.8136) (width 0.5) (layer "B.Cu") (net 21))
   (segment (start 94.0144 103.9713) (end 95.5766 105.5335) (width 0.5) (layer "B.Cu") (net 22))
   (segment (start 100.482 105.5335) (end 110.744 95.2715) (width 0.5) (layer "B.Cu") (net 22))
@@
   (segment (start 111.8321 88.1085) (end 105.6638 81.9402) (width 0.5) (layer "B.Cu") (net 23))
   (segment (start 113.284 88.1085) (end 111.8321 88.1085) (width 0.5) (layer "B.Cu") (net 23))
+  (segment (start 136.7972 66.6206) (end 124.7716 66.6206) (width 0.5) (layer "F.Cu") (net 24))
+  (segment (start 147.5951 95.6099) (end 147.5951 77.4185) (width 0.5) (layer "F.Cu") (net 24))
+  (segment (start 147.5951 77.4185) (end 136.7972 66.6206) (width 0.5) (layer "F.Cu") (net 24))
   (segment (start 130.9686 96.0882) (end 131.6942 96.8138) (width 0.5) (layer "F.Cu") (net 24))
   (segment (start 115.824 89.5604) (end 122.3518 96.0882) (width 0.5) (layer "F.Cu") (net 24))
-  (segment (start 131.6942 96.8138) (end 145.4253 96.8138) (width 0.5) (layer "F.Cu") (net 24))
-  (segment (start 147.5951 94.644) (end 147.5951 77.4185) (width 0.5) (layer "F.Cu") (net 24))
-  (segment (start 136.7972 66.6206) (end 124.7716 66.6206) (width 0.5) (layer "F.Cu") (net 24))
+  (segment (start 131.6942 96.8138) (end 146.3912 96.8138) (width 0.5) (layer "F.Cu") (net 24))
+  (segment (start 122.3518 96.0882) (end 130.9686 96.0882) (width 0.5) (layer "F.Cu") (net 24))
   (segment (start 121.8692 69.523) (end 121.8692 69.596) (width 0.5) (layer "F.Cu") (net 24))
-  (segment (start 147.5951 77.4185) (end 136.7972 66.6206) (width 0.5) (layer "F.Cu") (net 24))
-  (segment (start 145.4253 96.8138) (end 147.5951 94.644) (width 0.5) (layer "F.Cu") (net 24))
-  (segment (start 122.3518 96.0882) (end 130.9686 96.0882) (width 0.5) (layer "F.Cu") (net 24))
   (segment (start 124.7716 66.6206) (end 121.8692 69.523) (width 0.5) (layer "F.Cu") (net 24))
+  (segment (start 146.3912 96.8138) (end 147.5951 95.6099) (width 0.5) (layer "F.Cu") (net 24))
   (segment (start 140.897 75.9771) (end 138.664 78.2101) (width 0.5) (layer "F.Cu") (net 25))
   (segment (start 138.664 78.2101) (end 126.1201 78.2101) (width 0.5) (layer "F.Cu") (net 25))
